File: PCB/mini-devboard.kicad_pcb (KiCad board)
At the start: 2 copper layers, 19 x 56.4 mm, 16 parts, among them J1 USB_A, J2 Conn_02x05_Counter_Clockwise, SW1 SW_Push, U1 CH552G

Commit message: finishing touches
Parts:
- moved TP2 0.20 mm to (122.0, 89.0)
