File: PCB/mini-devboard.kicad_pcb (KiCad board)
At the start: 2 copper layers, 19 x 56.4 mm, 16 parts, among them J1 USB_A, J2 Conn_02x05_Counter_Clockwise, SW1 SW_Push, U1 CH552G

Commit message: changes i'm so tired
Connections:
- J2 pad 1: /P1.7 -> /P3.1
- J2 pad 2: /P1.6 -> /P3.0
- U1 pad 4: /P1.6 -> /Touch2
- U1 pad 5: /P1.7 -> /Touch1
- U1 pad 7: /Touch2 -> /P3.1
- U1 pad 8: /Touch1 -> /P3.0
Routing:
- net /P3.0: track 0.00 -> 32.3 mm
- net /P1.6: track 30.9 -> 0.00 mm
- net /P1.7: track 27.9 -> 0.00 mm
- net /P3.1: track 0.00 -> 27.3 mm
- net /Touch2: track 19.6 -> 21.7 mm
- net SCL: track 36.4 -> 37.6 mm
- net /Touch1: track 8.13 -> 9.16 mm
Other:
- board text added: "|======|======|======|======|======| | VBUS | +3V3 | SDA | SCL | P3.1 | |------|------|------|------|------| | GND | GND | P3.2 | P1.5 | P3.0 | |======|======|======|======|======|"
- board text removed: "|======|======|======|======|======| | VBUS | +3V3 | SDA | SCL | P1.7 | |------|------|------|------|------| | GND | GND | P3.2 | P1.5 | P1.6 | |======|======|======|======|======|"
