File: PCB/mini-devboard.kicad_sch (KiCad schematic)
At the start: 12 parts, among them J1 USB_A, J2 Conn_02x05_Counter_Clockwise, SW1 SW_Push, U1 CH552G

Commit message: make the pcb
Parts:
- added R4, R5: ?, Resistor_SMD:R_0805_2012Metric_Pad1.20x1.40mm_HandSolder, symbol Device:R
- added TP1, TP2: TestPoint_Alt, TestPoint:TestPoint_Pad_4.0x4.0mm, symbol Connector:TestPoint_Alt
- J2: symbol Connector_Generic:Conn_02x05_Counter_Clockwise -> Connector_Generic:Conn_02x05_Odd_Even
Connections:
- net +3V3: now also J2.7 (Pin_7), R4.2, R5.2; no longer J2.2 (Pin_2)
- net GND: now also J2.8 (Pin_8); no longer J2.9 (Pin_9)
- net P1.5: now also J2.4 (Pin_4); no longer J2.3 (Pin_3)
- net P3.2: now also J2.6 (Pin_6); no longer J2.8 (Pin_8)
- net SCL: now also J2.3 (Pin_3), R4.1; no longer J2.4 (Pin_4)
- net SDA: now also R5.1
- net VBUS: now also J2.9 (Pin_9); no longer J2.1 (Pin_1)
- net P1.6: now reaches U1.4 (P1.6)
- net P1.6: now also J2.2 (Pin_2)
- net P1.7: now reaches U1.5 (P1.7)
- net P1.7: now also J2.1 (Pin_1)
- net P3.0 renamed Touch1
- net Touch1: now also TP1.1; no longer J2.6 (Pin_6)
- net P3.1 renamed Touch2
- net Touch2: now also TP2.1; no longer J2.7 (Pin_7)

Commit message: organization
Other:
- note added: "I2C Pull Up"
- note added: "LEDs"
- note added: "MCU"
- moved on the sheet: D1, D2, R2, R3, R4, R5, TP1, TP2, U1

Commit message: changes i'm so tired
Parts:
- R4, R5: now not fitted
Connections:
- net Touch1: now also U1.5 (P1.7); no longer U1.8 (P3.0)
- net Touch2: now also U1.4 (P1.6); no longer U1.7 (P3.1)
- net P1.6 renamed P3.0
- net P3.0: now also U1.8 (P3.0); no longer U1.4 (P1.6)
- net P1.7 renamed P3.1
- net P3.1: now also U1.7 (P3.1); no longer U1.5 (P1.7)
Changed lines of the file:
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@@
-		)
-	)
-	(label "P1.7"
-		(at 50.8 81.28 180)
-		(effects
-			(font
-				(size 1.27 1.27)
-			)
-			(justify right bottom)
 		)
 	)
@@
 		)
 	)
-	(label "P1.6"
-		(at 63.5 81.28 0)
-		(effects
-			(font
-				(size 1.27 1.27)
-			)
-			(justify left bottom)
-		)
-	)
 	(label "D+"
 		(at 100.33 86.36 180)
@@
 	)
 	(label "Touch1"
-		(at 100.33 73.66 180)
-		(effects
-			(font
-				(size 1.27 1.27)
-			)
-			(justify right bottom)
+		(at 124.46 88.9 0)
+		(effects
+			(font
+				(size 1.27 1.27)
+			)
+			(justify left bottom)
 		)
 	)
@@
 		)
 	)
+	(label "P3.1"
+		(at 100.33 76.2 180)
+		(effects
+			(font
+				(size 1.27 1.27)
+			)
+			(justify right bottom)
+		)
+	)
 	(label "SCL"
 		(at 45.72 83.82 0)
@@
 	)
 	(label "Touch2"
-		(at 100.33 76.2 180)
+		(at 124.46 86.36 0)
+		(effects
+			(font
+				(size 1.27 1.27)
+			)
+			(justify left bottom)
+		)
+	)
+	(label "P3.0"
+		(at 100.33 73.66 180)
 		(effects
 			(font
@@
 			)
 			(justify right bottom)
-		)
-	)
-	(label "P1.6"
-		(at 124.46 86.36 0)
-		(effects
-			(font
-				(size 1.27 1.27)
-			)
-			(justify left bottom)
 		)
 	)
@@
 		)
 	)
+	(label "P3.1"
+		(at 50.8 81.28 180)
+		(effects
+			(font
+				(size 1.27 1.27)
+			)
+			(justify right bottom)
+		)
+	)
 	(label "SDA"
 		(at 100.33 83.82 180)
@@
 		)
 	)
-	(label "P1.7"
-		(at 124.46 88.9 0)
-		(effects
-			(font
-				(size 1.27 1.27)
-			)
-			(justify left bottom)
-		)
-	)
 	(label "SCL"
 		(at 179.07 38.1 0)
@@
 			)
 			(justify right bottom)
+		)
+	)
+	(label "P3.0"
+		(at 63.5 81.28 0)
+		(effects
+			(font
+				(size 1.27 1.27)
+			)
+			(justify left bottom)
 		)
 	)
@@
 		(on_board yes)
 		(in_pos_files yes)
-		(dnp no)
+		(dnp yes)
 		(fields_autoplaced yes)
 		(property "Reference" "R4"
@@
 		(on_board yes)
 		(in_pos_files yes)
-		(dnp no)
+		(dnp yes)
 		(fields_autoplaced yes)
 		(property "Reference" "R5"
